Commit message: add virtual joint

File: resources/soar/soar_spherized.urdf (robot description, URDF)
Before this commit: robot soar, 56 links, 55 joints
Links:
- added link virtual_link/theta
- added link virtual_link/x
- added link virtual_link/y
Joints:
- added joint virtual_joint/theta: type revolute, parent virtual_link/theta, child base_footprint, origin xyz=0 0 0.267 rpy=0 0 0, axis 0 0 1, limit lower=-6.283185307179586 upper=6.283185307179586 effort=50 velocity=4.71
- added joint virtual_joint/x: type prismatic, parent virtual_link/x, child virtual_link/y, origin xyz=0 0 0 rpy=0 0 0, axis 1 0 0, limit lower=-1.0 upper=1.0 effort=50 velocity=1.238
- added joint virtual_joint/y: type prismatic, parent virtual_link/y, child virtual_link/theta, origin xyz=0 0 0 rpy=0 0 0, axis 0 1 0, limit lower=-1.0 upper=1.0 effort=50 velocity=1.238

Commit message: update urdf

File: resources/soar/soar_spherized.urdf (robot description, URDF)
Before this commit: robot soar, 59 links, 58 joints
Links:
- link arm_left_finger: geometry collision sphere radius=0.01; collision sphere radius=0.01
- link arm_left_inner_knuckle: geometry collision sphere radius=0.01; collision sphere radius=0.01
- link arm_left_outer_knuckle: geometry collision sphere radius=0.01; collision sphere radius=0.01
- link arm_link1: geometry collision sphere radius=0.06; collision sphere radius=0.06
- link arm_link2: geometry collision sphere radius=0.053; collision sphere radius=0.053
- link arm_link3: geometry collision sphere radius=0.05; collision sphere radius=0.05
- link arm_link4: geometry collision sphere radius=0.052; collision sphere radius=0.052
- link arm_link5: geometry collision sphere radius=0.04; collision sphere radius=0.04
- link arm_link6: geometry collision sphere radius=0.04; collision sphere radius=0.04
- link arm_link7: geometry collision sphere radius=0.04; collision sphere radius=0.05
- link arm_link_base: geometry visual mesh filename=file:///home/ubuntu/ros/install/xarm_description/share/xarm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
- link arm_right_finger: geometry collision sphere radius=0.01; collision sphere radius=0.01
- link arm_right_inner_knuckle: geometry collision sphere radius=0.01; collision sphere radius=0.01
- link arm_right_outer_knuckle: geometry collision sphere radius=0.01; collision sphere radius=0.01
- link arm_xarm_gripper_base_link: geometry collision sphere radius=0.03; collision sphere radius=0.03
- link base_link: geometry collision sphere radius=0.05; collision sphere radius=0.05
- link front_caster_link: geometry collision sphere radius=0.047; collision sphere radius=0.047
- link hand_camera_mount_link: geometry visual mesh filename=file:///home/ubuntu/ros/install/soar_description/share/soar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
- link head_pan_link: geometry collision sphere radius=0.03; collision sphere radius=0.03
- link head_tilt_link: geometry collision sphere radius=0.03; collision sphere radius=0.03
- link power_connector_link: geometry visual mesh filename=file:///home/ubuntu/ros/install/soar_description/share/soar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
- link rear_caster_link: geometry collision sphere radius=0.047; collision sphere radius=0.047
- link torso_link: geometry collision sphere radius=0.07; collision sphere radius=0.07
- link wheel_left: geometry collision sphere radius=0.0569775; visual cylinder length=0.045 radius=0.0569775
- link wheel_right: geometry collision sphere radius=0.0569775; visual cylinder length=0.045 radius=0.0569775
Joints:
- joint virtual_joint/theta: origin xyz=0 0 0.267 rpy=0 0 0 -> xyz=0 0 0 rpy=0 0 0
